Commit message: Change RGB camera to  RGBD camera

File: catkin_ws/src/slam_project/urdf/udacity_bot.xacro (robot description, xacro)
@@ -175,4 +175,10 @@
     <parent link="chassis"/>
   </joint>
+  <link name="rgbd_frame"/>
+  <joint type="fixed" name="rgbd_frame_joint">
+    <origin xyz="0 0 0" rpy="-1.5707 0 -1.5707"/>
+    <child link="rgbd_frame"/>
+    <parent link="camera"/>
+  </joint>
   <link name="hokuyo">
     <visual name="visual">
